Commit message: Update simon-v2-0.urdf

File: simon-v2-0.urdf (robot description, URDF)
Before this commit: robot simon-v2-0, 10 links, 9 joints
Joints:
- joint joint_1: limit lower=-3.2 upper=3.2 effort=200 velocity=3 -> lower=-0.0867 upper=5.8579 effort=200 velocity=3
- joint joint_2: limit lower=-0.3621 upper=5.3019 effort=200 velocity=3 -> lower=-0.3621 upper=3.4556 effort=200 velocity=3
